File: hardware/epaper.kicad_pcb (KiCad board)
At the start: 2 copper layers, 65 x 30 mm, 56 parts, among them J1 download, J2 epaper, J3 USB_C_Receptacle_USB2.0, J4 BATT, J5 Speaker, J6 JTAG, Q1 DMG3404L, Q2 AO3401A, Q3 S8050, Q4 S8050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

Commit message: refactor: adjust file structure
Routing:
- net GND: vias 37 -> 54
